Commit message: Refactor comments for clarity in rover.urdf.xacro

File: description/rover.urdf.xacro (robot description, xacro)
@@ -1,5 +1,4 @@
 <?xml version="1.0"?>
 <robot xmlns:xacro="http://www.ros.org/wiki/xacro" name="urc_rover">
-  <!-- ==================== PROPERTIES ==================== -->
   <!-- All units: meters, kg, radians -->
   <!-- Chassis: simple box -->
@@ -10,7 +9,7 @@
   <!-- Wheels -->
   <xacro:property name="wheel_radius"     value="0.09525"/>   <!-- 3.75 in -->
-  <xacro:property name="wheel_width"      value="0.05"/>      <!-- 2 in, cosmetic -->
+  <xacro:property name="wheel_width"      value="0.05"/>
   <xacro:property name="wheel_mass"       value="0.5"/>
-  <xacro:property name="wheel_separation" value="0.8636"/>    <!-- 34 in center-to-center -->
+  <xacro:property name="wheel_separation" value="0.8636"/>    <!-- 34 in center to center -->
   <!-- Wheel Y offset from base_link center (half track width) -->
   <xacro:property name="wheel_y_offset" value="${wheel_separation / 2.0}"/>
@@ -21,5 +20,5 @@
   <!-- Chassis sits so wheel axles are at ground level (z=0 at ground) -->
   <xacro:property name="chassis_z_offset" value="${wheel_radius + chassis_height / 2.0}"/>
-  <!-- ==================== INERTIA MACROS ==================== -->
+  <!-- INERTIA MACROS -->
   <xacro:macro name="box_inertia" params="m x y z">
     <inertial>
@@ -38,5 +37,5 @@
     </inertial>
   </xacro:macro>
-  <!-- ==================== WHEEL MACRO ==================== -->
+  <!-- WHEEL MACRO -->
   <xacro:macro name="wheel" params="name x_pos y_pos">
     <link name="${name}_link">
@@ -65,5 +64,5 @@
     </joint>
   </xacro:macro>
-  <!-- ==================== LINKS & JOINTS ==================== -->
+  <!--  LINKS & JOINTS  -->
   <!-- base_link: at wheel-axle height, center of chassis footprint -->
   <link name="base_link">
@@ -106,5 +105,5 @@
   <xacro:wheel name="middle_left_wheel"  x_pos="${wheel_x_middle}" y_pos="${wheel_y_offset}"/>
   <xacro:wheel name="back_left_wheel"    x_pos="${wheel_x_back}"   y_pos="${wheel_y_offset}"/>
-  <!-- ==================== ROS2_CONTROL ==================== -->
+  <!-- ROS2_CONTROL -->
   <!--
     This block tells controller_manager to load SparkCanHardware and wire
